File: KicadJE_MoogVCF_1/KicadJE_Yousynth_MoogVCF.sch (KiCad schematic (older format))
At the start: 0 parts

Commit message: diff stage sch
Parts:
- added C?: C8, Capacitor_SMD:C_0805_2012Metric_Pad1.15x1.40mm_HandSolder, symbol Device:C
- added C? (x4): 100n, Capacitor_SMD:C_0805_2012Metric_Pad1.15x1.40mm_HandSolder, symbol Device:C
- added C? (x2): 10u, Capacitor_SMD:C_1206_3216Metric_Pad1.42x1.75mm_HandSolder, symbol Device:C
- added D? (x2): 1N1007, Diode_SMD:D_SOD-123, symbol Device:D
- added D? (x4): Zener, Diode_SMD:D_MiniMELF, symbol Device:D_Zener
- added H? (x2): 2,5mm, MountingHole:MountingHole_2.5mm_Pad_Via, symbol Mechanical:MountingHole
- added H? (x2): 2,2mm, MountingHole:MountingHole_2.2mm_M2_Pad_Via, symbol Mechanical:MountingHole
- added J?: In Gate, AJ-Dropbox-Kicad:PJ301SM, symbol Connector:AudioJack2_SwitchT
- added J?: Out Tom, AJ-Dropbox-Kicad:PJ301SM, symbol Connector:AudioJack2
- added J?: In_Accent, Connector_Audio:Jack_3.5mm_Ledino_KB3SPRS_Horizontal, symbol Connector:AudioJack2_SwitchT
- added P?: Doepfer_Power_10pin, Connectors_IDC:IDC-Header_2x05_Pitch2.54mm_Straight, symbol Eurorack:Doepfer_Power_10pin
- added Q? (x4): MMBT2222A, Package_TO_SOT_SMD:SOT-23_Handsoldering, symbol MMBT2222A:MMBT2222A
- added Q?: MMBT2907A, Package_TO_SOT_SMD:SOT-23_Handsoldering, symbol MMBT2907_:MMBT2907*
- added R?: 22R, Resistor_SMD:R_0805_2012Metric_Pad1.15x1.40mm_HandSolder, symbol Device:R
- added R?: 10k, Resistor_SMD:R_0805_2012Metric_Pad1.15x1.40mm_HandSolder, symbol Device:R
- added R? (x2): 270k, Resistor_SMD:R_0805_2012Metric_Pad1.15x1.40mm_HandSolder, symbol Device:R
- added R? (x2): 4k7, Resistor_SMD:R_0805_2012Metric_Pad1.15x1.40mm_HandSolder, symbol Device:R
- added R?: 1k, Resistor_SMD:R_0805_2012Metric_Pad1.15x1.40mm_HandSolder, symbol Device:R
- added R? (x2): 1K, Resistor_SMD:R_0805_2012Metric_Pad1.15x1.40mm_HandSolder, symbol Device:R
- added R? (x2): OPEN, Resistor_SMD:R_0805_2012Metric_Pad1.15x1.40mm_HandSolder, symbol Device:R
- added R?: 0R, Resistor_SMD:R_0805_2012Metric_Pad1.15x1.40mm_HandSolder, symbol Device:R
- added R?: 180R, Resistor_SMD:R_0805_2012Metric_Pad1.15x1.40mm_HandSolder, symbol Device:R
- added R?: 1k2, Resistor_SMD:R_0805_2012Metric_Pad1.15x1.40mm_HandSolder, symbol Device:R
- added TP?: Coupling, TestPoint:TestPoint_Pad_1.5x1.5mm, symbol Connector:TestPoint
- added U? (x3): TL072, AJ-Dropbox-Kicad:AJ_SO-8_5.3x6.2mm_P1.27mm, symbol Amplifier_Operational:TL072
Connections:
- net labels added: +12V, +12v, -12V, -12v, Coupling, GND, InAccent, InGate, OutVCF, PNP_B, PNP_E
- wire segments 0 -> 138
