File: KicadJE_MoogVCF_1/_autosave-KicadJE_MoogVCF_1.kicad_pcb (KiCad board)
At the start: 2 copper layers, 100 x 100 mm, 91 parts, among them J201 CV2, J202 Input, J203 CV1, J204 Out VCF, P201 Doepfer_Power_10pin, Q201 UMX1N, Q202 SS9014, Q203 SS9014, Q204 SS9014, Q205 SS9014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

Commit message: Placing components
Parts:
- added D209: Zener, Diode_SMD:D_MiniMELF, B.Cu at (22.7, 101.5)
- added D210: Zener, Diode_SMD:D_MiniMELF, B.Cu at (29.0, 101.5)
- added J205: Input, AJ-Dropbox-Kicad:PJ301SM, F.Cu at (59.8, 135.0)
- added R240: 1K, Resistor_SMD:R_0805_2012Metric_Pad1.15x1.40mm_HandSolder, B.Cu at (21.9, 98.4)
- added R241: OPEN, Resistor_SMD:R_0805_2012Metric_Pad1.15x1.40mm_HandSolder, B.Cu at (22.5, 105.3)
- added RV206: 50k_CV2, AJ-Dropbox-Kicad:Potentiometer_China_RK09_Single_Vertical_AJ, F.Cu at (52.2, 122.5)
- moved Q202 94.7 mm to (27.9, 19.2)
- moved Q207 88.5 mm to (34.8, 34.8)
- moved D208 58.2 mm to (-24.0, 103.6)
- moved H203 58.2 mm to (-20.8, 97.4)
- moved Q203 58.1 mm to (34.8, 19.2)
- moved Q211 56.0 mm to (0.75, 33.8)
- moved Q206 54.6 mm to (27.9, 34.7)
- moved Q201 54.4 mm to (31.3, 17.5), turned to 0 degrees
- moved Q212 53.7 mm to (0.75, 39.5)
- moved Q208 50.6 mm to (31.5, 36.2), turned to 180 degrees
- moved Q204 43.9 mm to (27.9, 27.5)
- moved RV201 43.1 mm to (87.2, 67.5), turned to 180 degrees
- moved Q205 37.1 mm to (34.8, 27.5)
- moved RV203 36.6 mm to (52.2, 107.5), turned to 0 degrees
- moved H204 27.4 mm to (-20.2, 91.0)
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Connections:
- J201 pad S: (no net) -> GND
- R221 pad 1: InAudio -> (no net)
- R234 pad 1: CV2 -> Net-(R234-Pad1)
