File: KicadJE_MoogVCF_1/_autosave-KicadJE_MoogVCF_1.kicad_pcb (KiCad board)
At the start: 2 copper layers, 100 x 100 mm, 99 parts, among them J201 CV2, J202 Input2, J203 CV1, J204 Out VCF, J205 Input1, P201 Doepfer_Power_10pin, Q201 UMX1N, Q202 SS9014, Q203 SS9014, Q204 SS9014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

Commit message: all components placed
Parts:
- added G***: LOGO, AJ:Johansen_engineering_logo_20mm, F.Cu at (79.0, 135.0)
Other:
- board text added: "06/10-2019"
- board text added: "JE - Moog VCF - Rev A"
- board text added: "MOOG VCF"
