File: KicadJE_MoogVCF_1/KicadJE_MoogVCF_1.kicad_pcb (KiCad board)
At the start: 2 copper layers, 100 x 100 mm, 99 parts, among them J201 CV2, J202 Input2, J203 CV1, J204 Out VCF, J205 Input1, P201 Doepfer_Power_10pin, Q201 UMX1N, Q202 SS9014, Q203 SS9014, Q204 SS9014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

Commit message: Moog VCF complete
Parts:
- added G***: LOGO, AJ:Johansen_engineering_logo_20mm, F.Cu at (79.0, 135.0)
Routing:
- net Net-(C211-Pad2): track 0.00 -> 63.4 mm
- net Net-(C213-Pad1): track 0.00 -> 52.0 mm, vias 0 -> 1
- net Net-(C212-Pad1): track 13.1 -> 59.8 mm
- net Net-(Q208-Pad5): track 0.00 -> 38.8 mm, vias 0 -> 2
- net +12V: track 99.8 -> 135.0 mm, vias 0 -> 2
- net CV1: track 8.47 -> 35.8 mm, vias 0 -> 2
- net Net-(Q206-Pad1): track 0.00 -> 23.9 mm, vias 0 -> 4
- net Net-(Q204-Pad1): track 0.00 -> 19.8 mm
- net /KicadJE_Yousynth_MoogVCF/PNP_B: track 48.2 -> 67.3 mm
- net Net-(Q202-Pad1): track 0.00 -> 18.4 mm
- net Net-(R211-Pad1): track 0.00 -> 16.3 mm
- net /KicadJE_Yousynth_MoogVCF/Coupling: track 0.00 -> 13.7 mm
- net Net-(R234-Pad1): track 0.00 -> 13.7 mm
- net -12V: track 96.4 -> 110.0 mm
- net Net-(Q208-Pad1): track 0.00 -> 11.9 mm
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Other:
- board text added: "06/10-2019"
- board text added: "JE - Moog VCF - Rev A"
- board text added: "MOOG VCF"
