File: KicadJE_MoogVCF_1/KicadJE_Yousynth_ADSR.sch (KiCad schematic (older format))
At the start: 51 parts

Commit message: ADSR sch done
Parts:
- added D?: 1N4148, Diode_SMD:D_SOD-123, symbol Device:D
- added R?: 100R, Resistor_SMD:R_0805_2012Metric_Pad1.15x1.40mm_HandSolder, symbol Device:R
- added R?: 1k, Resistor_SMD:R_0805_2012Metric_Pad1.15x1.40mm_HandSolder, symbol Device:R
- added U?: TL072, AJ-Dropbox-Kicad:AJ_SO-8_5.3x6.2mm_P1.27mm, symbol Amplifier_Operational:TL072
- RV?: value 50k_emphasis -> 1M Release
- RV?: value 50k_emphasis -> 1M Attack
Connections:
- wire segments 144 -> 164
Other:
- note added: "Fast"
- note added: "Slow"
- moved on the sheet: R?, RV?

Commit message: ADSR Routed
Parts:
- removed P?: Doepfer_Power_16pin, Connectors_IDC:IDC-Header_2x08_Pitch2.54mm_Straight, symbol Eurorack:Doepfer_Power_16pin
- removed Q? (x3): MMBT2222A, SOT23, symbol MMBT2222A:MMBT2222A
- added P301: Doepfer_Power_10pin, Connectors_IDC:IDC-Header_2x05_Pitch2.54mm_Straight, symbol Eurorack:Doepfer_Power_10pin
- added Q302, Q303, Q304: MMBT3904, Package_TO_SOT_SMD:SOT-23_Handsoldering, symbol MMBT2222A:MMBT2222A
- C306: renamed from C?; value 10u -> 10u_N/A
- Q301: renamed from Q?; value 2N7000 -> SI2302; footprint Package_TO_SOT_THT:TO-92_Inline -> Package_TO_SOT_SMD:SOT-23_Handsoldering; symbol Transistor_FET:2N7000 -> Transistor_FET:DMG2302U
- R304: renamed from R?; value 120R -> 120R_N/A
- SW301: renamed from SW?; footprint (none) -> AJ:Johansen_engineering_logo_20mm
- SW302: renamed from SW?; footprint (none) -> Button_Switch_THT:SW_PUSH_6mm
- gave numbers to parts that had none: 43
Connections:
- net labels removed: +5V
- wire segments 164 -> 167
