File: KicadJE_MoogVCF_1_revB/KicadJE_Yousynth_MoogVCF_revB.sch (KiCad schematic (older format))
At the start: 105 parts, among them J201 CV2, J202 Input2, J203 CV1, J204 Out VCF, J205 Input1, P201 Doepfer_Power_10pin, Q202 SS9014, Q203 SS9014, Q204 SS9014, Q205 SS9014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

Commit message: revb update
Parts:
- added C? (x2): 220n, Capacitor_SMD:C_0805_2012Metric_Pad1.15x1.40mm_HandSolder, symbol Device:C
Connections:
- net at Q?.5 (B), R227.2: now also C?.2
- net at Q?.2 (B), R226.2: now also C?.2
- net at C207.1, Q203.3 (C), Q?.4 (E): now also C?.1
- net at C207.2, Q202.3 (C), Q?.1 (E): now also C?.1
Other:
- note added: "Missing from RevA"
Changed lines of the file:
@@
 Wire Wire Line
 	8525 6100 8525 6200
-Connection ~ 8525 4375
-Wire Wire Line
-	8525 4375 8525 4450
 Wire Wire Line
 	5250 4375 5250 3750
@@
 Wire Wire Line
 	8050 5800 8250 5800
+Wire Wire Line
+	7500 5125 7500 4525
+Wire Wire Line
+	7500 4525 5625 4525
+Wire Wire Line
+	5625 4525 5625 1950
+Wire Wire Line
+	5625 1950 4800 1950
+Connection ~ 7500 5125
+Wire Wire Line
+	5750 1775 5750 4450
+Wire Wire Line
+	8875 4450 8875 5125
+Connection ~ 3475 1775
+Connection ~ 8875 5125
+Connection ~ 8525 4375
+Wire Wire Line
+	8525 4375 8525 4450
+Wire Wire Line
+	5750 4450 8875 4450
+$Comp
+L Device:C C?
+U 1 1 5E533F64
+P 4650 1775
+AR Path="/5D99B81E/5E533F64" Ref="C?"  Part="1"
+AR Path="/5D99B7BA/5E533F64" Ref="C?"  Part="1"
+F 0 "C?" V 4550 1825 50  0000 L CNN
+F 1 "220n" V 4600 1575 50  0000 L CNN
+F 2 "Capacitor_SMD:C_0805_2012Metric_Pad1.15x1.40mm_HandSolder" H 4688 1625 50  0001 C CNN
+F 3 "~" H 4650 1775 50  0001 C CNN
+	1    4650 1775
+	0    -1   -1   0
+$EndComp
+Wire Wire Line
+	4800 1775 5750 1775
+$Comp
+L Device:C C?
+U 1 1 5E5352A9
+P 4650 1950
+AR Path="/5D99B81E/5E5352A9" Ref="C?"  Part="1"
+AR Path="/5D99B7BA/5E5352A9" Ref="C?"  Part="1"
+F 0 "C?" V 4550 2000 50  0000 L CNN
+F 1 "220n" V 4600 1750 50  0000 L CNN
+F 2 "Capacitor_SMD:C_0805_2012Metric_Pad1.15x1.40mm_HandSolder" H 4688 1800 50  0001 C CNN
+F 3 "~" H 4650 1950 50  0001 C CNN
+	1    4650 1950
+	0    -1   -1   0
+$EndComp
+Wire Wire Line
+	4500 1950 3975 1950
+Wire Wire Line
+	3475 1775 4500 1775
+Text Notes 4900 1925 0    50   ~ 0
+Missing from RevA
 $EndSCHEMATC
