File: KicadJE_MoogVCF_1_revB/KicadJE_MoogVCF_1b.kicad_pcb (KiCad board)
At the start: 2 copper layers, 100 x 100 mm, 245 parts, among them J201 CV2, J202 Input2, J203 CV1, J204 Out VCF, J205 Input1, J301 ADSRGate, J302 ADSR, J401 CV, J402 Output, J403 VCA Out, J404 Input, P201 Doepfer_Power_10pin, P301 Doepfer_Power_10pin, P401 Doepfer_Power_10pin, Q201 UMX1N, Q202 SS9014, Q203 SS9014, Q204 SS9014, Q205 SS9014, Q206 SS9014, Q207 SS9014, Q208 UMX1N, Q209 UMX1N, Q210 UMX1N, Q211 SS9014, Q212 SS9015, Q301 SI2302, Q302 MMBT3904, Q303 MMBT3904, Q304 MMBT3904, Q401 UMX1N, Q402 SS9014, SW301 SW_DPDT_x2, SW302 Gate, U201 TL072, U301 TL072, U302 TLC555, U401 TL072, U402 TL074

Commit message: Faceplate for Moog Filter
Parts:
- added REF**: MountingHole_Eurorack3, AJ:MountingHole_Eurorack3, F.Cu at (213.5, 161.0)
- added REF**: MountingHole_Eurorack3, AJ:MountingHole_Eurorack3, F.Cu at (186.5, 161.0)
- added REF**: MountingHole_Eurorack3, AJ:MountingHole_Eurorack3, F.Cu at (213.5, 39.0)
- added REF**: MountingHole_Eurorack3, AJ:MountingHole_Eurorack3, F.Cu at (186.5, 39.0)
Other:
- board size 100 x 100 mm -> 170 x 128 mm

Commit message: Wavefolder Faceplate
Parts:
- added G***: LOGO, AJ:Johansen_engineering_logo_25mm_front_neg5, B.Cu at (200.0, 46.0)
- added G***: LOGO, AJ:Johansen_engineering_logo_25mm_front_neg5, B.Cu at (268.0, 46.0)
- added G***: LOGO, AJ:Johansen_engineering_soldermask_20mm, F.Cu at (267.5, 161.0)
- added G***: LOGO, AJ:Johansen_engineering_soldermask_20mm, F.Cu at (200.0, 161.0)
- added REF**: 6,3mm inner, AJ:Jack_3m5, F.Cu at (277.0, 140.0)
- added REF**: MountingHole_Eurorack3, AJ:MountingHole_Eurorack3, F.Cu at (281.0, 39.0)
- added REF**: MountingHole_Eurorack3, AJ:MountingHole_Eurorack3, F.Cu at (254.0, 39.0)
- added REF**: 6,3mm inner pot, AJ:Pot_6m3_scale1, F.Cu at (209.5, 70.0)
- added REF**: 6,3mm inner pot, AJ:Pot_6m3_scale1, F.Cu at (190.0, 70.0)
- added REF**: 6,3mm inner pot, AJ:Pot_6m3_scale1, F.Cu at (190.0, 105.0)
- added REF**: 6,3mm inner pot, AJ:Pot_6m3_scale1, F.Cu at (190.0, 120.0)
- added REF**: 6,3mm inner, AJ:Jack_3m5, F.Cu at (189.5, 135.0)
- added REF**: 6,3mm inner, AJ:Jack_3m5, F.Cu at (209.5, 105.0)
- added REF**: 6,3mm inner, AJ:Jack_3m5, F.Cu at (209.5, 120.0)
- added REF**: 6,3mm inner, AJ:Jack_3m5, F.Cu at (209.5, 145.0)
- added REF**: 6,3mm inner pot, AJ:Pot_6m3_scale1, F.Cu at (257.5, 70.0)
- added REF**: 6,3mm inner, AJ:Jack_3m5, F.Cu at (189.5, 145.0)
- added REF**: 6,3mm inner, AJ:Jack_3m5, F.Cu at (257.0, 130.0)
- added REF**: 6,3mm inner, AJ:Jack_3m5, F.Cu at (277.0, 130.0)
- added REF**: 6,3mm inner, AJ:Jack_3m5, F.Cu at (257.0, 140.0)
- added REF**: 6,3mm inner pot, AJ:Pot_6m3_scale1, F.Cu at (277.0, 70.0)
- added REF**: 6,3mm inner pot, AJ:Pot_6m3_scale1, F.Cu at (257.5, 95.0)
- added REF**: MountingHole_Eurorack3, AJ:MountingHole_Eurorack3, F.Cu at (281.0, 161.0)
- added REF**: MountingHole_Eurorack3, AJ:MountingHole_Eurorack3, F.Cu at (254.0, 161.0)
Connections:
- REF** pad 1: (no net) -> GND (x4)
Other:
- board size 170 x 128 mm -> 237.5 x 128 mm
- board text added: "CV1"
- board text added: "CV2"
- board text added: "E"
- board text added: "F"
- board text added: "In1"
- board text added: "In2"
- board text added: "M-VCF"
- board text added: "Out"
- board text added: "Range"
- board text added: "Shape"
- board text added: "VCA"
- board text added: "W-FLD"
